File: NARA.sch (KiCad schematic (older format))
At the start: 122 parts

Commit message: Update schematic
Parts:
- removed C? (x2): C_0037, DVB_Capacitors_Ceramic:C_0603, symbol C_0037
- removed P?: TOF_LF, zhonx_lib:Conn_Serial_Zhonx, symbol Samtec_UART
- removed P?: Samtec_UART, zhonx_lib:Conn_Serial_Zhonx, symbol Samtec_UART
- removed P?: TOF_LD, zhonx_lib:Conn_Serial_Zhonx, symbol Samtec_UART
- removed P?: TOF_LS, zhonx_lib:Conn_Serial_Zhonx, symbol Samtec_UART
- removed P?: TOF_RF, zhonx_lib:Conn_Serial_Zhonx, symbol Samtec_UART
- removed P?: TOF_RD, zhonx_lib:Conn_Serial_Zhonx, symbol Samtec_UART
- removed P?: TOF_RS, zhonx_lib:Conn_Serial_Zhonx, symbol Samtec_UART
- removed Q? (x3): Q_0004, DVB_SOT:SOT_23, symbol Q_0004
- removed R? (x3): R_0002, DVB_Resistors:R_0402, symbol R_0002
- removed R? (x2): R_0033, DVB_Resistors:R_0402, symbol R_0033
- removed R? (x2): R_0105, DVB_Resistors:R_0402, symbol R_0105
- removed U?: STM32H743VITx, LQFP100, symbol STM32H743VITx
- removed U? (x2): QRE1113GR, zhonx_lib:QRE1113GR, symbol QRE1113GR
- added C25: C_0001, DVB_Capacitors_Ceramic:C_0402, symbol C_0001
- added C26, C39, C40: C_0037, DVB_Capacitors_Ceramic:C_0603, symbol C_0037
- added C27, C32: C_0043, DVB_Capacitors_Ceramic:C_0402, symbol C_0043
- added C28, C44: C_0002, DVB_Capacitors_Ceramic:C_0402, symbol C_0002
- added C29, C31, C34, C35, C36: C_0007, DVB_Capacitors_Ceramic:C_1206, symbol C_0007
- added C30, C33: C_0045, DVB_Capacitors_Ceramic:C_0402, symbol C_0045
- added D10, D5, D6, D7, D8, D9: D_0001, DVB_LED:LED_0603-red, symbol D_0001
- added K10: TOF_LD, n.c, symbol CONN_01X04
- added K11: TOF_LS, n.c, symbol CONN_01X04
- added K12: TOF_RF, n.c, symbol CONN_01X04
- added K13: TOF_RD, n.c, symbol CONN_01X04
- added K14: TOF_RS, n.c, symbol CONN_01X04
- added K15: UART, n.c, symbol CONN_01X04
- added K2: PW_MOT, n.c, symbol CONN_01X02
- added K3: PROG, n.c, symbol CONN_01X03
- added K4: OLED, n.c, symbol CONN_01X04
- added K9: TOF_LF, n.c, symbol CONN_01X04
- added L2: L_0010, DVB_Inductors:L_0603, symbol L_0010
- added Q1, Q9: Q_0004, DVB_SOT:SOT_23, symbol Q_0004
- added R23: R_0118, DVB_Resistors:R_0402, symbol R_0118
- added R24: R_0015, DVB_Resistors:R_0402, symbol R_0015
- added R25, R26, R27, R28: R_0104, DVB_Resistors:R_0402, symbol R_0104
- added R37, R46, R8: R_0002, DVB_Resistors:R_0402, symbol R_0002
- added R38: R_0076, DVB_Resistors:R_0603, symbol R_0076
- added R49, R50: R_0033, DVB_Resistors:R_0402, symbol R_0033
- added R55, R56: R_0105, DVB_Resistors:R_0402, symbol R_0105
- added SP1: SP_0001, DVB_Buzzers:SP_KSSG-5x5x3, symbol SP_0001
- added SW2: KMR223G, Buttons_Switches_SMD:SW_SPST_KMR2, symbol SW_PUSH
- added U11, U12: QRE1113GR, zhonx_lib:QRE1113GR, symbol QRE1113GR
- added U7: STM32H743VITx, LQFP100, symbol STM32H743VITx
- added XO1: XO_0001-RESCUE-HM3, DVB_Clock:XO_8Z, symbol XO_0001-RESCUE-HM3
- gave numbers to parts that had none: 100
Connections:
- net labels added: BEEPER, LED1, LED2, LED3, LED4, LINE_ADC_L1, LINE_ADC_L2, LINE_ADC_R1, LINE_ADC_R2, LINE_EN, PW_3V_EN, PW_5V_EN
- net labels removed: LINE_IN_L1, LINE_IN_L2, LINE_IN_R1, LINE_IN_R2, LINE_OUT_L1, LINE_OUT_L2, LINE_OUT_R1, LINE_OUT_R2, PW_EN
- wire segments 159 -> 144
- no-connect marks 3 -> 27
Other:
- moved on the sheet: C1, C10, C11, C12, C13, C14, C15, C16, C17, C2, C20, C21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

Commit message: First schematic version
Parts:
- K2: fabricant (none) -> n.c
Changed lines of the file:
@@
 F 4 "K_" V 3850 850 50  0001 C CNN "sIdProduct"
 F 5 "n.c" V 3925 850 50  0001 C CNN "details"
-F 6 "n.c" V 4000 850 50  0001 C CNN "fabricant
-"
+F 6 "n.c" V 4000 850 50  0001 C CNN "fabricant"
 	1    3525 850
 	-1   0    0    1

Commit message: Update schematic create nara.lib
Parts:
- removed C18, C19: C_, DVB_Capacitors_Ceramic:C_0603, symbol C_0012
- removed C4, C5, C7, C8: C_, DVB_Capacitors_Tantalum:CP_EIA-7343-31, symbol C_0020
- removed K1: K_0034, DVB_Connectors:K_CTB93HE-2, symbol K_0034
- removed K5, K7: K_, DVB_Connectors:K_PicoSPOX-3, symbol K_
- removed SW1, SW2: KMR223G, Buttons_Switches_SMD:SW_SPST_KMR2, symbol SW_PUSH
- removed U13: U_0049, DVB_SOT:SOT_143, symbol U_0049
- removed U2: U_, DVB_SOT:SOT_23-5, symbol U_0085
- added C18, C19: C_220nF, DVB_Capacitors_Ceramic:C_0603, symbol C_220nF
- added C4, C5, C7, C8: C_47uF, DVB_Capacitors_Tantalum:CP_EIA-7343-31, symbol C_47uF
- added C45: C_470nF, DVB_Capacitors_Ceramic:C_0402, symbol C_470nF
- added D11: D_0001, DVB_LED:LED_0603-red, symbol D_0001
- added K1: K_KK-41791-02, Connectors_Molex:Molex_KK-41791-02_02x3.96mm_Straight, symbol K_KK-41791-02
- added K5, K7: K_PicoSPOX-3, DVB_Connectors:K_PicoSPOX-3, symbol K_PicoSPOX-3
- added R57: R_0104, DVB_Resistors:R_0402, symbol R_0104
- added R58, R61: R_0033, DVB_Resistors:R_0402, symbol R_0033
- added R59, R60: R_0105, DVB_Resistors:R_0402, symbol R_0105
- added R62, R63, R64, R65, R66, R67: R_0111, DVB_Resistors:R_0402, symbol R_0111
- added SW1, SW2, SW3, SW4: SW_KMR2, Buttons_Switches_SMD:SW_SPST_KMR2, symbol SW_KMR2
- added U2: U_AP2204K-5.0TRG1, DVB_SOT:SOT_23-5, symbol U_AP2204K-5.0TRG1
- K15: footprint n.c -> Pin_Headers:Pin_Header_Straight_1x04_Pitch2.54mm
- K2: footprint n.c -> Pin_Headers:Pin_Header_Straight_1x02_Pitch2.54mm; details n.c -> Jumper
- K3: footprint n.c -> Pin_Headers:Pin_Header_Straight_1x03_Pitch2.54mm
Connections:
- net labels added: USER_SW1, USER_SW2
- wire segments 144 -> 164
- no-connect marks 27 -> 25
Other:
- note added: "6 axis Accelerometer and Gyroscope"
- note added: "Beeper"
- note added: "Bluetooth"
- note added: "Display"
- note added: "Encoder Power"
- note added: "Floor Sensors"
- note added: "Fuel Gauge"
- note added: "Left Motor Driver"
- note added: "Main Power"
- note added: "Microcontroller"
- note added: "Prog"
- note added: "Push Button Controller"
- note added: "Reset Button"
- note added: "Right Motor Driver"
- note added: "TOF Sensors"
- note added: "User Buttons"
- note added: "User LED"
- moved on the sheet: C37, C38, C39, C40, C41, C42, C43, D10, D7, D8, D9, K10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

Commit message: Add NARA_Lib.pretty
Parts:
- removed K10: TOF_LD, n.c, symbol CONN_01X04
- removed K11: TOF_LS, n.c, symbol CONN_01X04
- removed K12: TOF_RF, n.c, symbol CONN_01X04
- removed K13: TOF_RD, n.c, symbol CONN_01X04
- removed K14: TOF_RS, n.c, symbol CONN_01X04
- removed K4: OLED, n.c, symbol CONN_01X04
- removed K9: TOF_LF, n.c, symbol CONN_01X04
- added K10: TOF_LD, NARA_Lib:GYVL53L0X, symbol GYVL53L0X
- added K11: TOF_LS, NARA_Lib:GYVL53L0X, symbol GYVL53L0X
- added K12: TOF_LR, NARA_Lib:GYVL53L0X, symbol GYVL53L0X
- added K13: TOF_RD, NARA_Lib:GYVL53L0X, symbol GYVL53L0X
- added K14: TOF_RS, NARA_Lib:GYVL53L0X, symbol GYVL53L0X
- added K16: OLED_128x32, NARA_Lib:OLED_128x32, symbol OLED_128x32
- added K9: TOF_LF, NARA_Lib:GYVL53L0X, symbol GYVL53L0X
Connections:
- net +3.3V: now also K16.2 (Vcc)
- net GND: now also K10.3 (GND), K11.3 (GND), K12.3 (GND), K13.3 (GND), K14.3 (GND), K16.1 (GND), K9.3 (GND)
- net OLED_SCL: now also K16.3 (SCL)
- net OLED_SDA: now also K16.4 (SDA)
- net TOF_L_SCL: now also K10.2 (SCL), K11.2 (SCL), K9.2 (SCL)
- net TOF_L_SDA: now also K10.1 (SDA), K11.1 (SDA), K9.1 (SDA)
- net TOF_R_SCL: now also K12.2 (SCL), K13.2 (SCL), K14.2 (SCL)
- net TOF_R_SDA: now also K12.1 (SDA), K13.1 (SDA), K14.1 (SDA)
- net at Q2.3 (D): now also K9.4 (VIN)
- net at Q5.3 (D): now also K12.4 (VIN)
- net at Q3.3 (D): now also K10.4 (VIN)
- net at Q6.3 (D): now also K13.4 (VIN)
- net at Q4.3 (D): now also K11.4 (VIN)
- net at Q7.3 (D): now also K14.4 (VIN)
Changed lines of the file:
@@
 Sheet 1 1
 Title "NARA"
-Date "2018-04-08"
-Rev "0.0.4"
+Date "2018-04-09"
+Rev "0.0.5"
 Comp "PACABOT"
 Comment1 ""
@@
 U 1 1 5AC70AEB
 P 2375 1275
-F 0 "U3" H 2625 975 50  0000 C CNN
+F 0 "U3" H 2625 925 50  0000 C CNN
 F 1 "LTC2944" H 2375 725 50  0001 C CNN
 F 2 "Housings_DFN_QFN:DFN-8-1EP_3x3mm_Pitch0.5mm" H 2375 625 50  0001 C CNN
@@
 $EndComp
 $Comp
-L CONN_01X04 K4
-U 1 1 5ACE8D30
-P 14025 2375
-F 0 "K4" H 14025 2625 50  0000 C CNN
-F 1 "OLED" V 14125 2375 50  0000 C CNN
-F 2 "n.c" V 14275 2375 50  0001 C CNN
-F 3 "n.c" V 14200 2375 50  0001 C CNN
-F 4 "K_" V 14350 2375 50  0001 C CNN "sIdProduct"
-F 5 "n.c" V 14425 2375 50  0001 C CNN "details"
-F 6 "n.c" V 14500 2375 50  0001 C CNN "fabricant"
-	1    14025 2375
-	1    0    0    1
-$EndComp
-$Comp
 L GND #PWR0125
 U 1 1 5ACE9376
@@
 $EndComp
 $Comp
-L CONN_01X04 K9
-U 1 1 5ACEA343
-P 9150 7750
-F 0 "K9" H 9150 8000 50  0000 C CNN
-F 1 "TOF_LF" V 9250 7750 50  0000 C CNN
-F 2 "n.c" V 9400 7750 50  0001 C CNN
-F 3 "n.c" V 9325 7750 50  0001 C CNN
-F 4 "K_" V 9475 7750 50  0001 C CNN "sIdProduct"
-F 5 "n.c" V 9550 7750 50  0001 C CNN "details"
-F 6 "n.c" V 9625 7750 50  0001 C CNN "fabricant"
-	1    9150 7750
-	1    0    0    1
-$EndComp
-$Comp
-L CONN_01X04 K12
-U 1 1 5ACEC006
-P 10500 7750
-F 0 "K12" H 10500 8000 50  0000 C CNN
-F 1 "TOF_RF" V 10600 7750 50  0000 C CNN
-F 2 "n.c" V 10750 7750 50  0001 C CNN
-F 3 "n.c" V 10675 7750 50  0001 C CNN
-F 4 "K_" V 10825 7750 50  0001 C CNN "sIdProduct"
-F 5 "n.c" V 10900 7750 50  0001 C CNN "details"
-F 6 "n.c" V 10975 7750 50  0001 C CNN "fabricant"
-	1    10500 7750
-	1    0    0    1
-$EndComp
-$Comp
-L CONN_01X04 K13
-U 1 1 5ACEC83A
-P 10500 9025
-F 0 "K13" H 10500 9275 50  0000 C CNN
-F 1 "TOF_RD" V 10600 9025 50  0000 C CNN
-F 2 "n.c" V 10750 9025 50  0001 C CNN
-F 3 "n.c" V 10675 9025 50  0001 C CNN
-F 4 "K_" V 10825 9025 50  0001 C CNN "sIdProduct"
-F 5 "n.c" V 10900 9025 50  0001 C CNN "details"
-F 6 "n.c" V 10975 9025 50  0001 C CNN "fabricant"
-	1    10500 9025
-	1    0    0    1
-$EndComp
-$Comp
-L CONN_01X04 K10
-U 1 1 5ACECE58
-P 9150 9025
-F 0 "K10" H 9150 9275 50  0000 C CNN
-F 1 "TOF_LD" V 9250 9025 50  0000 C CNN
-F 2 "n.c" V 9400 9025 50  0001 C CNN
-F 3 "n.c" V 9325 9025 50  0001 C CNN
-F 4 "K_" V 9475 9025 50  0001 C CNN "sIdProduct"
-F 5 "n.c" V 9550 9025 50  0001 C CNN "details"
-F 6 "n.c" V 9625 9025 50  0001 C CNN "fabricant"
-	1    9150 9025
-	1    0    0    1
-$EndComp
-$Comp
-L CONN_01X04 K11
-U 1 1 5ACED45E
-P 9150 10300
-F 0 "K11" H 9150 10550 50  0000 C CNN
-F 1 "TOF_LS" V 9250 10300 50  0000 C CNN
-F 2 "n.c" V 9400 10300 50  0001 C CNN
-F 3 "n.c" V 9325 10300 50  0001 C CNN
-F 4 "K_" V 9475 10300 50  0001 C CNN "sIdProduct"
-F 5 "n.c" V 9550 10300 50  0001 C CNN "details"
-F 6 "n.c" V 9625 10300 50  0001 C CNN "fabricant"
-	1    9150 10300
-	1    0    0    1
-$EndComp
-$Comp
-L CONN_01X04 K14
-U 1 1 5ACEDEE8
-P 10500 10300
-F 0 "K14" H 10500 10550 50  0000 C CNN
-F 1 "TOF_RS" V 10600 10300 50  0000 C CNN
-F 2 "n.c" V 10750 10300 50  0001 C CNN
-F 3 "n.c" V 10675 10300 50  0001 C CNN
-F 4 "K_" V 10825 10300 50  0001 C CNN "sIdProduct"
-F 5 "n.c" V 10900 10300 50  0001 C CNN "details"
-F 6 "n.c" V 10975 10300 50  0001 C CNN "fabricant"
-	1    10500 10300
-	1    0    0    1
-$EndComp
-$Comp
 L CONN_01X04 K15
 U 1 1 5ACEFB05
@@
 	5750 3725 5750 3825
 Connection ~ 5750 3775
+$Comp
+L GYVL53L0X K9
+U 1 1 5ACB394B
+P 9150 7750
+F 0 "K9" H 9150 8000 50  0000 C CNN
+F 1 "TOF_LF" V 9350 7600 50  0000 C CNN
+F 2 "NARA_Lib:GYVL53L0X" H 9150 7125 50  0001 C CNN
+F 3 "n.c" H 9150 7425 50  0001 C CNN
+F 4 "K_" H 9150 7350 50  0001 C CNN "sIdProduct"
+F 5 "n.c" H 9150 7275 50  0001 C CNN "details"
+F 6 "n.c" H 9150 7200 50  0001 C CNN "fabricant"
+	1    9150 7750
+	1    0    0    -1
+$EndComp
+$Comp
+L GYVL53L0X K12
+U 1 1 5ACB481F
+P 10500 7750
+F 0 "K12" H 10500 8000 50  0000 C CNN
+F 1 "TOF_LR" V 10700 7600 50  0000 C CNN
+F 2 "NARA_Lib:GYVL53L0X" H 10500 7125 50  0001 C CNN
+F 3 "n.c" H 10500 7425 50  0001 C CNN
+F 4 "K_" H 10500 7350 50  0001 C CNN "sIdProduct"
+F 5 "n.c" H 10500 7275 50  0001 C CNN "details"
+F 6 "n.c" H 10500 7200 50  0001 C CNN "fabricant"
+	1    10500 7750
+	1    0    0    -1
+$EndComp
+$Comp
+L GYVL53L0X K13
+U 1 1 5ACB518B
+P 10500 9025
+F 0 "K13" H 10500 9275 50  0000 C CNN
+F 1 "TOF_RD" V 10700 8875 50  0000 C CNN
+F 2 "NARA_Lib:GYVL53L0X" H 10500 8400 50  0001 C CNN
+F 3 "n.c" H 10500 8700 50  0001 C CNN
+F 4 "K_" H 10500 8625 50  0001 C CNN "sIdProduct"
+F 5 "n.c" H 10500 8550 50  0001 C CNN "details"
+F 6 "n.c" H 10500 8475 50  0001 C CNN "fabricant"
+	1    10500 9025
+	1    0    0    -1
+$EndComp
+$Comp
+L GYVL53L0X K10
+U 1 1 5ACB5F1C
+P 9150 9025
+F 0 "K10" H 9150 9275 50  0000 C CNN
+F 1 "TOF_LD" V 9350 8875 50  0000 C CNN
+F 2 "NARA_Lib:GYVL53L0X" H 9150 8400 50  0001 C CNN
+F 3 "n.c" H 9150 8700 50  0001 C CNN
+F 4 "K_" H 9150 8625 50  0001 C CNN "sIdProduct"
+F 5 "n.c" H 9150 8550 50  0001 C CNN "details"
+F 6 "n.c" H 9150 8475 50  0001 C CNN "fabricant"
+	1    9150 9025
+	1    0    0    -1
+$EndComp
+$Comp
+L GYVL53L0X K11
+U 1 1 5ACB67F9
+P 9150 10300
+F 0 "K11" H 9150 10550 50  0000 C CNN
+F 1 "TOF_LS" V 9350 10150 50  0000 C CNN
+F 2 "NARA_Lib:GYVL53L0X" H 9150 9675 50  0001 C CNN
+F 3 "n.c" H 9150 9975 50  0001 C CNN
+F 4 "K_" H 9150 9900 50  0001 C CNN "sIdProduct"
+F 5 "n.c" H 9150 9825 50  0001 C CNN "details"
+F 6 "n.c" H 9150 9750 50  0001 C CNN "fabricant"
+	1    9150 10300
+	1    0    0    -1
+$EndComp
+$Comp
+L GYVL53L0X K14
+U 1 1 5ACB6EFC
+P 10500 10300
+F 0 "K14" H 10500 10550 50  0000 C CNN
+F 1 "TOF_RS" V 10700 10150 50  0000 C CNN
+F 2 "NARA_Lib:GYVL53L0X" H 10500 9675 50  0001 C CNN
+F 3 "n.c" H 10500 9975 50  0001 C CNN
+F 4 "K_" H 10500 9900 50  0001 C CNN "sIdProduct"
+F 5 "n.c" H 10500 9825 50  0001 C CNN "details"
+F 6 "n.c" H 10500 9750 50  0001 C CNN "fabricant"
+	1    10500 10300
+	1    0    0    -1
+$EndComp
+$Comp
+L OLED_128x32 K16
+U 1 1 5ACBACF6
+P 14025 2375
+F 0 "K16" H 14025 2625 50  0000 C CNN
+F 1 "OLED_128x32" H 14575 2625 50  0000 C CNN
+F 2 "NARA_Lib:OLED_128x32" H 14075 2025 50  0001 C CNN
+F 3 "n.c" H 14075 2125 50  0001 C CNN
+F 4 "K_" H 14075 1925 50  0001 C CNN "sIdProduct"
+F 5 "n.c" H 14075 1825 50  0001 C CNN "details"
+F 6 "n.c" H 14075 1725 50  0001 C CNN "fabricant"
+	1    14025 2375
+	1    0    0    -1
+$EndComp
 $EndSCHEMATC

Commit message: Update footprints, prepare to place composants
Parts:
- removed U1: U_0065, DVB_SSOP:MSOP_16-EP_3x4_P0.5, symbol U_0065
- removed XO1: XO_0001-RESCUE-HM3, DVB_Clock:XO_8Z, symbol XO_0001-RESCUE-HM3
- added U1: U_LT8610ABIMSE-3.3, DVB_SSOP:MSOP_16-1EP_3x4_P0.5, symbol U_LT8610ABIMSE-3.3
- added XO1: XO_8Z-16, DVB_Clock:XO_8Z, symbol XO_8Z-16
- K5, K7: footprint DVB_Connectors:K_PicoSPOX-3 -> NARA_Lib:K_PicoSPOX-3
- U10, U11, U12, U9: footprint zhonx_lib:QRE1113GR -> NARA_Lib:QRE1113GR
- U4, U5: footprint (none) -> NARA_Lib:PowerSO-20
- U6: footprint zhonx_lib:LTC2955 -> TO_SOT_Packages_SMD:SOT-23-8
- U7: footprint LQFP100 -> Housings_QFP:LQFP-100_14x14mm_Pitch0.5mm
- U8: footprint (none) -> Housings_DFN_QFN:QFN-24-1EP_4x4mm_Pitch0.5mm
Connections:
- net +3.3V: now also U1.14 (BIAS), U1.16 (Vout)
- net +BATT: now also U1.5 (Vin), U1.6 (Vin)
- net GND: now also U1.1 (SYNC), U1.17 (GND), U1.8 (GND), XO1.2, XO1.4
- net PW_3V_EN: now also U1.4 (EN/UV)
- net at C11.2, L1.1: now also U1.10 (SW), U1.11 (SW), U1.9 (SW)
- net at C11.1: now also U1.12 (BST)
- net at C6.1: now also U1.13 (INTVcc)
- net at C2.1: now also U1.2 (TR/SS)
- net at R17.1: now also U1.3 (RT)
- net at C27.2, U7.12 (PH0/RCC_OSC_IN): now also XO1.1
- net at C32.1, U7.13 (PH1/RCC_OSC_OUT): now also XO1.3
Other:
- moved on the sheet: C41, C42, C43, C45

Commit message: First components placement, Autoroute in progress
Parts:
- removed C20: C_0001, DVB_Capacitors_Ceramic:C_0402, symbol C_0001
- removed C27, C32: C_0043, DVB_Capacitors_Ceramic:C_0402, symbol C_0043
- removed C31, C34, C35, C36: C_0007, DVB_Capacitors_Ceramic:C_1206, symbol C_0007
- removed D10, D6, D7, D8, D9: D_0001, DVB_LED:LED_0603-red, symbol D_0001
- removed F1: F_001, DVB_F:F-OMNI-BLOCK, symbol F_001
- removed K1: K_KK-41791-02, Connectors_Molex:Molex_KK-41791-02_02x3.96mm_Straight, symbol K_KK-41791-02
- removed K15: UART, Pin_Headers:Pin_Header_Straight_1x04_Pitch2.54mm, symbol CONN_01X04
- removed K16: OLED_128x32, NARA_Lib:OLED_128x32, symbol OLED_128x32
- removed K2: PW_MOT, Pin_Headers:Pin_Header_Straight_1x02_Pitch2.54mm, symbol CONN_01X02
- removed R24: R_0015, DVB_Resistors:R_0402, symbol R_0015
- removed R25, R26, R27, R28: R_0104, DVB_Resistors:R_0402, symbol R_0104
- removed R51, R52: R_0003, DVB_Resistors:R_0402, symbol R_0003
- removed R58, R61: R_0033, DVB_Resistors:R_0402, symbol R_0033
- removed R59, R60: R_0105, DVB_Resistors:R_0402, symbol R_0105
- removed SW1, SW2, SW3, SW4: SW_KMR2, Buttons_Switches_SMD:SW_SPST_KMR2, symbol SW_KMR2
- removed XO1: XO_8Z-16, DVB_Clock:XO_8Z, symbol XO_8Z-16
- added C31, C34, C35, C36: C_0002, DVB_Capacitors_Ceramic:C_0402, symbol C_0002
- added F1: FUSE, DVB_F:F_1206, symbol FUSE
- added K1: BATT, DVB_Connectors:Pin_Header_Straight_1x02_Pitch2.54mm, symbol CONN_01X02
- added K2: K_FPC_52435-2471, DVB_Connectors:K_FPC_52435-2471, symbol K_FPC_52435-2471
- added SW1, SW2: SW_SKQG, DVB_Buttons:SPST_SKQG, symbol SW_SKQG
- K12: value TOF_LR -> TOF_RF
- K3: footprint Pin_Headers:Pin_Header_Straight_1x03_Pitch2.54mm -> DVB_Connectors:Pin_Header_Straight_1x03_Pitch2.54mm
- U3: footprint Housings_DFN_QFN:DFN-8-1EP_3x3mm_Pitch0.5mm -> DVB_QFN_DFN:DFN_8-1EP_3x3mm_P0.5mm
- U6: footprint TO_SOT_Packages_SMD:SOT-23-8 -> DVB_SOT:SOT_23-8
- U7: footprint Housings_QFP:LQFP-100_14x14mm_Pitch0.5mm -> DVB_QFP:LQFP-100_14x14mm_Pitch0.5mm
- U8: footprint Housings_DFN_QFN:QFN-24-1EP_4x4mm_Pitch0.5mm -> DVB_QFN_DFN:QFN-24-1EP_4x4mm_Pitch0.5mm
Connections:
- net +HBAT is gone; now on net +BATT: C10.1, C4.1, C5.1, C7.1, C8.1, C9.1, D1.2 (A), D2.2 (A), U4.12 (VS), U4.9 (VS), U5.12 (VS), U5.9 (VS)
- net +3.3V: now also C31.2, C34.2, C35.2, C36.2, K2.22, K2.23, K2.24
- net +BATT: now also C21.2; no longer C21.1
- net BLUETOOTH_RX: now also K2.14
- net BLUETOOTH_TX: now also K2.13
- net GND: now also C21.1, C31.1, C34.1, C35.1, C36.1, K1.1 (P1), K2.1 (P1), K2.12, K2.19, K2.3, K2.9, SW1.2, SW2.1; no longer C21.2
- net LED1: now also K2.15
- net LED2: now also K2.16
- net LED3: now also K2.17
- net LED4: now also K2.18
- net OLED_SCL: now also K2.10
- net OLED_SDA: now also K2.11
- net SWCLK: now also K2.7
- net SWDIO: now also K2.8
- net USER_SW1: now also K2.4
- net USER_SW2: now also K2.5
- net ~RESET: now also K2.6, SW2.2
- net at R18.2, U3.8 (SENSE-): now also F1.1
- net EXT_ADC1: now reaches U7.17 (PC2)
- net EXT_ADC1: now also K2.21
- net EXT_ADC2: now reaches U7.18 (PC3)
- net EXT_ADC2: now also K2.20
- net SW_PW: now reaches U6.5 (PB)
- net SW_PW: now also K2.2 (P2), SW1.1
- new net: F1.2, K1.2 (P2)
Other:
- note added: "Extention connector"
- note removed: "Bluetooth"
- note removed: "Display"
- note removed: "User Buttons"
- note removed: "User LED"
- moved on the sheet: C17, C22, C23, C25, C37, C38, C39, C40, C41, C42, C43, C45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

Commit message: Change EdgeCuts for TOF sensors, adapt power trace lengh
Parts:
- removed R19, R20: R_0093, DVB_Resistors:R_1206, symbol R_0093
- removed R21, R22: R_0015, DVB_Resistors:R_0402, symbol R_0015
Connections:
- net GND: now also U4.19 (SENSE2), U4.2 (SENSE1), U5.19 (SENSE2), U5.2 (SENSE1)
- net MOT_L_SENSE: no longer names the net of U7.33 (PC5)
- net MOT_R_SENSE: no longer names the net of U7.34 (PB0)
- no-connect marks 25 -> 27
