File: NARA.sch (KiCad schematic (older format))
At the start: 140 parts, among them K1 BATT, K10 TOF_LD, K11 TOF_LS, K12 TOF_RF, K13 TOF_RD, K14 TOF_RS, K2 K_FPC_52435-2471, K3 PROG, K5 K_PicoSPOX-3, K6 K_0002, K7 K_PicoSPOX-3, K8 K_0002, K9 TOF_LF, Q1 Q_0004, Q2 Q_0007, Q3 Q_0007, Q4 Q_0007, Q5 Q_0007, Q6 Q_0007, Q7 Q_0007, Q8 Q_0004, Q9 Q_0004, SW1 SW_SKQG, SW2 SW_SKQG, U1 U_LT8610ABIMSE-3.3, U10 QRE1113GR, U11 QRE1113GR, U12 QRE1113GR, U2 U_AP2204K-5.0TRG1, U3 LTC2944, U4 L6234, U5 L6234, U6 LTC2955TS8-1, U7 STM32H743VITx, U8 ICM-20689, U9 QRE1113GR

Commit message: New v1.1.0, add jtag Connector and main led
Parts:
- removed K3: PROG, DVB_Connectors:Pin_Header_Straight_1x03_Pitch2.54mm, symbol CONN_01X03
- added D6: D_0001, DVB_LED:LED_0603-red, symbol D_0001
- added K3: DVB_JTAG-10, NARA_Lib:FTSH-105-XX-X-DV, symbol DVB_JTAG-10
- added R19: R_0104, DVB_Resistors:R_0402, symbol R_0104
- K1: footprint DVB_Connectors:Pin_Header_Straight_1x02_Pitch2.54mm -> NARA_Lib:Pin_Header_Straight_1x02_Pitch3mm
- K10: value TOF_LD -> TOF_RD
- K11: value TOF_LS -> TOF_RS
- K12: value TOF_RF -> TOF_LF
- K13: value TOF_RD -> TOF_LD
- K14: value TOF_RS -> TOF_LS
- K9: value TOF_LF -> TOF_RF
Connections:
- net +3.3V: now also K3.10 (3.3V), K3.9 (3.3V), R19.1
- net BLUETOOTH_RX: now also K3.8 (RX)
- net BLUETOOTH_TX: now also K3.6 (TX)
- net GND: now also K3.1 (GND), K3.2 (GND)
- net LED1: now also D6.1 (K)
- net LINE_ADC_L1: now also R55.2, U11.3 (C), U7.28 (PA4); no longer R53.2, U7.15 (PC0), U9.3 (C)
- net LINE_ADC_L2: now also R56.2, U12.3 (C), U7.29 (PA5); no longer R54.2, U10.3 (C), U7.16 (PC1)
- net LINE_ADC_R1: now also R53.2, U7.15 (PC0), U9.3 (C); no longer R55.2, U11.3 (C), U7.28 (PA4)
- net LINE_ADC_R2: now also R54.2, U10.3 (C), U7.16 (PC1); no longer R56.2, U12.3 (C), U7.29 (PA5)
- net MOT_L_EN1: now also R10.2, U5.8 (EN1), U7.31 (PA7); no longer R9.2, U4.8 (EN1), U7.38 (PE8)
- net MOT_L_EN2: now also R13.2, U5.3 (EN2), U7.53 (PB14); no longer R12.2, U4.3 (EN2), U7.40 (PE10)
- net MOT_L_EN3: now also R16.2, U5.13 (EN3), U7.54 (PB15); no longer R15.2, U4.13 (EN3), U7.42 (PE12)
- net MOT_L_HALL1: now also R36.2, U7.59 (PD12); no longer R33.2, U7.22 (PA0)
- net MOT_L_HALL2: now also R35.2, U7.60 (PD13); no longer R32.2, U7.23 (PA1)
- net MOT_L_HALL3: now also R34.2, U7.61 (PD14); no longer R31.2, U7.24 (PA2)
- net MOT_L_IN1: now also R2.2, U5.7 (IN1), U7.63 (PC6); no longer R1.2, U4.7 (IN1), U7.39 (PE9)
- net MOT_L_IN2: now also R4.2, U5.4 (IN2), U7.64 (PC7); no longer R3.2, U4.4 (IN2), U7.41 (PE11)
- net MOT_L_IN3: now also R6.2, U5.14 (IN3), U7.65 (PC8); no longer R5.2, U4.14 (IN3), U7.43 (PE13)
- net MOT_L_PHASE_A_BRO: now also K7.3 (P3), U5.6 (OUT1); no longer K5.3 (P3), U4.6 (OUT1)
- net MOT_L_PHASE_B_ORA: now also K7.2 (P2), U5.5 (OUT2); no longer K5.2 (P2), U4.5 (OUT2)
- net MOT_L_PHASE_C_YEL: now also K7.1 (P1), U5.15 (OUT3); no longer K5.1 (P1), U4.15 (OUT3)
- net MOT_R_EN1: now also R9.2, U4.8 (EN1), U7.38 (PE8); no longer R10.2, U5.8 (EN1), U7.31 (PA7)
- net MOT_R_EN2: now also R12.2, U4.3 (EN2), U7.40 (PE10); no longer R13.2, U5.3 (EN2), U7.53 (PB14)
- net MOT_R_EN3: now also R15.2, U4.13 (EN3), U7.42 (PE12); no longer R16.2, U5.13 (EN3), U7.54 (PB15)
- net MOT_R_HALL1: now also R33.2, U7.22 (PA0); no longer R36.2, U7.59 (PD12)
- net MOT_R_HALL2: now also R32.2, U7.23 (PA1); no longer R35.2, U7.60 (PD13)
- net MOT_R_HALL3: now also R31.2, U7.24 (PA2); no longer R34.2, U7.61 (PD14)
- net MOT_R_IN1: now also R1.2, U4.7 (IN1), U7.39 (PE9); no longer R2.2, U5.7 (IN1), U7.63 (PC6)
- net MOT_R_IN2: now also R3.2, U4.4 (IN2), U7.41 (PE11); no longer R4.2, U5.4 (IN2), U7.64 (PC7)
- net MOT_R_IN3: now also R5.2, U4.14 (IN3), U7.43 (PE13); no longer R6.2, U5.14 (IN3), U7.65 (PC8)
- net MOT_R_PHASE_A_BRO: now also K5.3 (P3), U4.6 (OUT1); no longer K7.3 (P3), U5.6 (OUT1)
- net MOT_R_PHASE_B_ORA: now also K5.2 (P2), U4.5 (OUT2); no longer K7.2 (P2), U5.5 (OUT2)
- net MOT_R_PHASE_C_YEL: now also K5.1 (P1), U4.15 (OUT3); no longer K7.1 (P1), U5.15 (OUT3)
- net SWCLK: now also K3.5 (SWD-CLK)
- net SWDIO: now also K3.3 (SWD-IO)
- net TOF_EN_LD: now also Q6.1 (G), R43.2, U7.84 (PD3); no longer Q3.1 (G), R40.2, U7.87 (PD6)
- net TOF_EN_LF: now also Q5.1 (G), R42.2, U7.85 (PD4); no longer Q2.1 (G), R39.2, U7.88 (PD7)
- net TOF_EN_LS: now also Q7.1 (G), R44.2, U7.83 (PD2); no longer Q4.1 (G), R41.2, U7.86 (PD5)
- net TOF_EN_RD: now also Q3.1 (G), R40.2, U7.87 (PD6); no longer Q6.1 (G), R43.2, U7.84 (PD3)
- net TOF_EN_RF: now also Q2.1 (G), R39.2, U7.88 (PD7); no longer Q5.1 (G), R42.2, U7.85 (PD4)
- net TOF_EN_RS: now also Q4.1 (G), R41.2, U7.86 (PD5); no longer Q7.1 (G), R44.2, U7.83 (PD2)
- net TOF_L_SCL: now also K12.2 (SCL), K13.2 (SCL), K14.2 (SCL), R67.2, U7.67 (PA8); no longer K10.2 (SCL), K11.2 (SCL), K9.2 (SCL), R65.2, U7.46 (PB10)
- net TOF_L_SDA: now also K12.1 (SDA), K13.1 (SDA), K14.1 (SDA), R66.1, U7.66 (PC9); no longer K10.1 (SDA), K11.1 (SDA), K9.1 (SDA), R64.1, U7.47 (PB11)
- net TOF_R_SCL: now also K10.2 (SCL), K11.2 (SCL), K9.2 (SCL), R65.2, U7.46 (PB10); no longer K12.2 (SCL), K13.2 (SCL), K14.2 (SCL), R67.2, U7.67 (PA8)
- net TOF_R_SDA: now also K10.1 (SDA), K11.1 (SDA), K9.1 (SDA), R64.1, U7.47 (PB11); no longer K12.1 (SDA), K13.1 (SDA), K14.1 (SDA), R66.1, U7.66 (PC9)
- net ~RESET: now also K3.4 (~tRST)
- new net: D6.2 (A), R19.2
- no-connect marks 27 -> 28
Other:
- note added: "Main LED"
