File: NARA.kicad_pcb (KiCad board)
At the start: 4 copper layers, 93.9 x 42.4 mm, 150 parts, among them K1 BATT, K10 TOF_RD, K11 TOF_RS, K12 TOF_LF, K13 TOF_LD, K14 TOF_LS, K2 K_FPC_52435-2471, K3 DVB_JTAG-10, K5 K_PicoSPOX-3, K6 K_0002, K7 K_PicoSPOX-3, K8 K_0002, K9 TOF_RF, Q1 Q_0004, Q2 Q_0007, Q3 Q_0007, Q4 Q_0007, Q5 Q_0007, Q6 Q_0007, Q7 Q_0007, Q8 Q_0004, Q9 Q_0004, SW1 SW_SKQG, SW2 SW_SKQG, U1 U_LT8610ABIMSE-3.3, U10 QRE1113GR, U11 QRE1113GR, U12 QRE1113GR, U2 U_AP2204K-5.0TRG1, U3 LTC2944, U4 L6234, U5 L6234, U6 LTC2955TS8-1, U7 STM32H743VITx, U8 ICM-20689, U9 QRE1113GR

Commit message: Update Gerbers (clean errors for Eurocircuit)
Routing:
- net +3.3V: track 361.3 -> 359.5 mm
- net +5V: track 43.8 -> 45.2 mm
- net Net-(C15-Pad2): vias 2 -> 1
- net +BATT: vias 22 -> 21

Commit message: Mouve debug connector
Parts:
- moved G*** 10.2 mm to (135.0, 103.0)
- moved K3 9.73 mm to (125.0, 104.5)
- moved G*** 0.65 mm to (130.8, 98.2)
Routing:
- net +3.3V: track 359.5 -> 370.2 mm
- net /SWCLK: track 54.6 -> 64.9 mm
- net /BLUETOOTH_TX: track 45.4 -> 55.6 mm
- net /SWDIO: track 51.1 -> 61.1 mm
- net /BLUETOOTH_RX: track 44.3 -> 54.2 mm
- net GND: track 847.2 -> 850.6 mm, vias 92 -> 91
- net /~RESET: track 50.2 -> 51.3 mm, vias 2 -> 3

Commit message: Change PCB sensors footprint
Routing:
- net /TOF_R_SDA: track 78.6 -> 76.2 mm
- net GND: track 850.6 -> 848.7 mm
- net /TOF_L_SCL: track 73.5 -> 72.7 mm
