File: NARA.kicad_pcb (KiCad board)
At the start: 4 copper layers, 93.9 x 42.4 mm, 150 parts, among them K1 BATT, K10 TOF_RD, K11 TOF_RS, K12 TOF_LF, K13 TOF_LD, K14 TOF_LS, K2 K_FPC_52435-2471, K3 DVB_JTAG-10, K5 K_PicoSPOX-3, K6 K_0002, K7 K_PicoSPOX-3, K8 K_0002, K9 TOF_RF, Q1 Q_0004, Q2 Q_0007, Q3 Q_0007, Q4 Q_0007, Q5 Q_0007, Q6 Q_0007, Q7 Q_0007, Q8 Q_0004, Q9 Q_0004, SW1 SW_SKQG, SW2 SW_SKQG, U1 U_LT8610ABIMSE-3.3, U10 QRE1113GR, U11 QRE1113GR, U12 QRE1113GR, U2 U_AP2204K-5.0TRG1, U3 LTC2944, U4 L6234, U5 L6234, U6 LTC2955TS8-1, U7 STM32H743VITx, U8 ICM-20689, U9 QRE1113GR

Commit message: In this version, we trust
Routing:
- net GND: track 848.6 -> 871.2 mm, vias 91 -> 93
- net +3.3V: track 370.6 -> 371.4 mm
- net /TOF_R_SCL: track 79.9 -> 79.1 mm
- net /TOF_L_SDA: track 73.9 -> 73.3 mm
Other:
- board text removed: "+"
